Commit message: Drop geometry that no eye can reach, measured instead of listed
The export carries 399 visual instances; some sit entirely inside the body.
Instead of a hand-kept whitelist, tools/visibility_bake.py ray-casts the whole
assembly (Open3D/Embree, 32 directions, 512x512, two door poses) and records
how many views each instance wins. 40 instances never win a pixel.

- tools/visibility_bake.py: the bake, writes docs/visibility.json (136 KB)
- visual_overrides.json: keep/drop exceptions, empty by default
- urdf_reduce.py: drops the <visual> of those instances per pose-verified key;
  mass and inertia stay in the link, so the total stays 14.412 kg
- urdf_verify.py: the 40 missing instances must be exactly the baked ones
- docs: what was measured, and the honest number — hiding buys 5.4 % of the
  triangles, the remaining 94.6 % is visible shell

File: urdf/pib.control.urdf (robot description, URDF)
Before this commit: robot pib, 49 links, 48 joints
Links:
- link a81_motor_shaft: geometry collision mesh filename=package://pib/meshes/A01_Face.glb scale=1 1 1; collision mesh filename=package://pib/meshes/A02_Face_neck_clamp.glb scale=1 1 1
- link c09_central_rotator_connector: geometry collision mesh filename=package://pib/meshes/C09_Central_rotator_connector.glb scale=1 1 1; collision mesh filename=package://pib/meshes/C18R_Forearm_distal_lock_right.glb scale=1 1 1
- link c09_central_rotator_connector_1: geometry collision mesh filename=package://pib/meshes/C09_Central_rotator_connector.glb scale=1 1 1; collision mesh filename=package://pib/meshes/C31_Elbow_shaft_motor.glb scale=1 1 1
- link c09_central_rotator_connector_2: geometry collision mesh filename=package://pib/meshes/C09_Central_rotator_connector.glb scale=1 1 1; collision mesh filename=package://pib/meshes/C31_Elbow_shaft_motor.glb scale=1 1 1
- link c09_central_rotator_connector_3: geometry collision mesh filename=package://pib/meshes/C09_Central_rotator_connector.glb scale=1 1 1; collision mesh filename=package://pib/meshes/C18L_Forearm_distal_lock_left.glb scale=1 1 1
- link c25_forearm_disc_bottom: geometry collision mesh filename=package://pib/meshes/C25_Forearm_disc_bottom.glb scale=1 1 1; collision mesh filename=package://pib/meshes/C30_Forearm_bar.glb scale=1 1 1
- link c25_forearm_disc_bottom_1: geometry collision mesh filename=package://pib/meshes/C30_Forearm_bar.glb scale=1 1 1; visual mesh filename=package://pib/meshes/C30_Forearm_bar.glb scale=1 1 1
- link c36_elbow_lower_shell: geometry collision mesh filename=package://pib/meshes/C33_Elbow_motor_flange.glb scale=1 1 1; collision mesh filename=package://pib/meshes/C36_Elbow_lower_shell.glb scale=1 1 1
- link c64_motor_axis_cap_inner_shoulder: geometry collision mesh filename=package://pib/meshes/C64_Motor_Axis_Cap_Inner_Shoulder.glb scale=1 1 1; collision mesh filename=package://pib/meshes/C65_Bracket_Outer_Shoulder.glb scale=1 1 1
- link c64_motor_axis_cap_inner_shoulder_1: geometry collision mesh filename=package://pib/meshes/C64_Motor_Axis_Cap_Inner_Shoulder.glb scale=1 1 1; collision mesh filename=package://pib/meshes/C65_Bracket_Outer_Shoulder.glb scale=1 1 1
- link c69_inner_part_outer_shoulder: geometry collision mesh filename=package://pib/meshes/C68_Inner_Ring_Outer_Shoulder.glb scale=1 1 1; collision mesh filename=package://pib/meshes/C69_Inner_Part_Outer_Shoulder.glb scale=1 1 1
- link c69_inner_part_outer_shoulder_1: geometry collision mesh filename=package://pib/meshes/C68_Inner_Ring_Outer_Shoulder.glb scale=1 1 1; collision mesh filename=package://pib/meshes/C69_Inner_Part_Outer_Shoulder.glb scale=1 1 1
- link root: geometry collision mesh filename=package://pib/meshes/A75_L_Neck_Left.glb scale=1 1 1; collision mesh filename=package://pib/meshes/A75_R_Neck_Right.glb scale=1 1 1

Commit message: Decide part by part what the model shows
121 parts are now listed in visual_overrides.json drop, 160 kept explicitly;
41 families were walked with the owner, 49 always-visible families were kept
automatically because they appear in every one of the 32 views.

Effect on the shipped model: 2,404,010 -> 1,575,930 triangles (-34 %), mesh
payload 57.0 -> 37.4 MB, 355 -> 171 visual/collision elements. Mass unchanged
(14.412 kg), all four verification tests pass.

Consequence the owner accepted: the silhouette is open where the dropped
parts were part of the shell (servo scaffolds on the upper arms, power holder,
forearm bars, hinge plates). tools/families.py restore <family> brings any of
them back.

File: urdf/pib.control.urdf (robot description, URDF)
Before this commit: robot pib, 49 links, 48 joints
Links:
- link a71_inner_part: geometry collision mesh filename=package://pib/meshes/A72_Top_part.glb scale=1 1 1; collision mesh filename=package://pib/meshes/A73_Cover_neck.glb scale=1 1 1
- link b44_electronics_back: geometry collision mesh filename=package://pib/meshes/B44_Electronics_back.glb scale=1 1 1; visual mesh filename=package://pib/meshes/B44_Electronics_back.glb scale=1 1 1
- link b46_power_back: geometry collision mesh filename=package://pib/meshes/B46_Power_back.glb scale=1 1 1; visual mesh filename=package://pib/meshes/B46_Power_back.glb scale=1 1 1
- link c09_central_rotator_connector: geometry collision mesh filename=package://pib/meshes/C18R_Forearm_distal_lock_right.glb scale=1 1 1; collision mesh filename=package://pib/meshes/C19R_Forearm_distal_top_right.glb scale=1 1 1
- link c09_central_rotator_connector_1: geometry collision mesh filename=package://pib/meshes/C31_Elbow_shaft_motor.glb scale=1 1 1; collision mesh filename=package://pib/meshes/C32_Elbow_axis_cable.glb scale=1 1 1
- link c09_central_rotator_connector_2: geometry collision mesh filename=package://pib/meshes/C31_Elbow_shaft_motor.glb scale=1 1 1; collision mesh filename=package://pib/meshes/C32_Elbow_axis_cable.glb scale=1 1 1
- link c09_central_rotator_connector_3: geometry collision mesh filename=package://pib/meshes/C18L_Forearm_distal_lock_left.glb scale=1 1 1; collision mesh filename=package://pib/meshes/C19L_Forearm_distal_top_left.glb scale=1 1 1
- link c25_forearm_disc_bottom: geometry 
- link c25_forearm_disc_bottom_1: geometry 
- link c36_elbow_lower_shell: geometry collision mesh filename=package://pib/meshes/C36_Elbow_lower_shell.glb scale=1 1 1; collision mesh filename=package://pib/meshes/C37_Elbow_rotator_bracket.glb scale=1 1 1
- link c36_elbow_lower_shell_1: geometry collision mesh filename=package://pib/meshes/C36_Elbow_lower_shell.glb scale=1 1 1; collision mesh filename=package://pib/meshes/C37_Elbow_rotator_bracket.glb scale=1 1 1
- link c64_motor_axis_cap_inner_shoulder: geometry collision mesh filename=package://pib/meshes/C65_Bracket_Outer_Shoulder.glb scale=1 1 1; collision mesh filename=package://pib/meshes/C66_Cap_Front_Outer_Shoulder.glb scale=1 1 1
- link c64_motor_axis_cap_inner_shoulder_1: geometry collision mesh filename=package://pib/meshes/C65_Bracket_Outer_Shoulder.glb scale=1 1 1; collision mesh filename=package://pib/meshes/C66_Cap_Front_Outer_Shoulder.glb scale=1 1 1
- link c69_inner_part_outer_shoulder: geometry collision mesh filename=package://pib/meshes/C69_Inner_Part_Outer_Shoulder.glb scale=1 1 1; collision mesh filename=package://pib/meshes/C70_Shell_Outer_Shoulder.glb scale=1 1 1
- link c69_inner_part_outer_shoulder_1: geometry collision mesh filename=package://pib/meshes/C69_Inner_Part_Outer_Shoulder.glb scale=1 1 1; collision mesh filename=package://pib/meshes/C70_Shell_Outer_Shoulder.glb scale=1 1 1
- link d01_l_palm_left: geometry collision mesh filename=package://pib/meshes/D01_L_Palm_left.glb scale=1 1 1; collision mesh filename=package://pib/meshes/D11_L_Bearing_enclosure_left.glb scale=1 1 1
- link d01_r_palm_right: geometry collision mesh filename=package://pib/meshes/D01_R_Palm_right.glb scale=1 1 1; collision mesh filename=package://pib/meshes/D11_R_Bearing_enclosure_right.glb scale=1 1 1
- link d13_l_thumb_rotator_left: geometry collision mesh filename=package://pib/meshes/D13_L_Thumb_rotator_left.glb scale=1 1 1; visual mesh filename=package://pib/meshes/D13_L_Thumb_rotator_left.glb scale=1 1 1
- link d13_r_thumb_rotator_right: geometry collision mesh filename=package://pib/meshes/D13_R_Thumb_rotator_right.glb scale=1 1 1; visual mesh filename=package://pib/meshes/D13_R_Thumb_rotator_right.glb scale=1 1 1
- link d52_finger_proximal: geometry collision mesh filename=package://pib/meshes/D52_Finger_proximal.glb scale=1 1 1; collision mesh filename=package://pib/meshes/D60_Proximal_skin.glb scale=1 1 1
- link d52_finger_proximal_1: geometry collision mesh filename=package://pib/meshes/D52_Finger_proximal.glb scale=1 1 1; collision mesh filename=package://pib/meshes/D60_Proximal_skin.glb scale=1 1 1
- link d52_finger_proximal_2: geometry collision mesh filename=package://pib/meshes/D52_Finger_proximal.glb scale=1 1 1; collision mesh filename=package://pib/meshes/D60_Proximal_skin.glb scale=1 1 1
- link d52_finger_proximal_3: geometry collision mesh filename=package://pib/meshes/D52_Finger_proximal.glb scale=1 1 1; collision mesh filename=package://pib/meshes/D60_Proximal_skin.glb scale=1 1 1
- link d52_finger_proximal_4: geometry collision mesh filename=package://pib/meshes/D52_Finger_proximal.glb scale=1 1 1; collision mesh filename=package://pib/meshes/D60_Proximal_skin.glb scale=1 1 1
- link d52_finger_proximal_5: geometry collision mesh filename=package://pib/meshes/D52_Finger_proximal.glb scale=1 1 1; collision mesh filename=package://pib/meshes/D60_Proximal_skin.glb scale=1 1 1
- link d52_finger_proximal_6: geometry collision mesh filename=package://pib/meshes/D52_Finger_proximal.glb scale=1 1 1; collision mesh filename=package://pib/meshes/D60_Proximal_skin.glb scale=1 1 1
- link d52_finger_proximal_7: geometry collision mesh filename=package://pib/meshes/D52_Finger_proximal.glb scale=1 1 1; collision mesh filename=package://pib/meshes/D60_Proximal_skin.glb scale=1 1 1
- link root: geometry collision mesh filename=package://pib/meshes/A75_L_Neck_Left.glb scale=1 1 1; collision mesh filename=package://pib/meshes/A75_R_Neck_Right.glb scale=1 1 1
